Commit message: WIP gz sim integration

File: roarm/urdf/roarm.xacro (robot description, xacro)
@@ -1,4 +1,5 @@
 <?xml version="1.0"?>
-<robot name="physics">
+<robot xmlns:xacro="http://www.ros.org/wiki/xacro">
+  <xacro:include filename="inertial_macros.xacro"/>
   <material name="gray">
     <color rgba="0.8 0.8 0.8 1"/>
@@ -15,4 +16,13 @@
       <material name="gray"/>
     </visual>
+    <collision>
+      <geometry>
+        <mesh filename="package://roarm/meshes/base.stl"/>
+      </geometry>
+      <origin rpy="0 0 0" xyz="0 0 0"/>
+    </collision>
+    <xacro:inertial_box mass="0.5" x="0.05" y="0.05" z="0.05">
+      <origin xyz="0 0 0" rpy="0 0 0"/>
+    </xacro:inertial_box>
   </link>
   <link name="l1_link">
@@ -24,4 +34,13 @@
       <material name="white"/>
     </visual>
+    <collision>
+      <geometry>
+        <mesh filename="package://roarm/meshes/L1.stl"/>
+      </geometry>
+      <origin rpy="0 0 0" xyz="0 0 0"/>
+    </collision>
+    <xacro:inertial_cylinder mass="0.5" radius="0.03" length="0.05">
+      <origin xyz="0 0 0" rpy="0 0 0"/>
+    </xacro:inertial_cylinder>
   </link>
   <link name="l2_link">
@@ -33,4 +52,13 @@
       <material name="white"/>
     </visual>
+    <collision>
+      <geometry>
+        <mesh filename="package://roarm/meshes/L2.stl"/>
+      </geometry>
+      <origin rpy="0 0 0" xyz="0 0 -0.03796"/>
+    </collision>
+    <xacro:inertial_cylinder mass="0.5" radius="0.03" length="0.05">
+      <origin xyz="0 0 0" rpy="0 0 0"/>
+    </xacro:inertial_cylinder>
   </link>
   <link name="l3_link">
@@ -42,4 +70,13 @@
       <material name="white"/>
     </visual>
+    <collision>
+      <geometry>
+        <mesh filename="package://roarm/meshes/L3.stl"/>
+      </geometry>
+      <origin rpy="0 0 0" xyz="-0.03 0 -0.27477"/>
+    </collision>
+    <xacro:inertial_cylinder mass="0.5" radius="0.03" length="0.05">
+      <origin xyz="0 0 0" rpy="0 0 0"/>
+    </xacro:inertial_cylinder>
   </link>
   <link name="l4_link">
@@ -51,4 +88,13 @@
       <material name="white"/>
     </visual>
+    <collision>
+      <geometry>
+        <mesh filename="package://roarm/meshes/L4.stl"/>
+      </geometry>
+      <origin rpy="0 0 0" xyz="-0.03 0 -0.49076"/>
+    </collision>
+    <xacro:inertial_cylinder mass="0.5" radius="0.03" length="0.05">
+      <origin xyz="0 0 0" rpy="0 0 0"/>
+    </xacro:inertial_cylinder>
   </link>
   <joint name="base_to_L1" type="revolute">

Commit message: Update inertia and get ros2 control working in gz sim

File: roarm/urdf/roarm.xacro (robot description, xacro)
@@ -1,5 +1,4 @@
 <?xml version="1.0"?>
 <robot xmlns:xacro="http://www.ros.org/wiki/xacro">
-  <xacro:include filename="inertial_macros.xacro"/>
   <material name="gray">
     <color rgba="0.8 0.8 0.8 1"/>
@@ -8,4 +7,6 @@
     <color rgba="1 1 1 1"/>
   </material>
+  <!--For now, set the inertial values according to here https://github.com/waveshareteam/roarm_ws_em0-->
+  <!--The current values are for the gripper layout roarm m2-->
   <link name="base_link">
     <visual>
@@ -22,7 +23,18 @@
       <origin rpy="0 0 0" xyz="0 0 0"/>
     </collision>
-    <xacro:inertial_box mass="0.5" x="0.05" y="0.05" z="0.05">
-      <origin xyz="0 0 0" rpy="0 0 0"/>
-    </xacro:inertial_box>
+    <inertial>
+      <origin
+        xyz="0.00373847392098165 -1.52445893424664E-10 0.0264265327292804"
+        rpy="0 0 0" />
+      <mass
+        value="0.326392759093976" />
+      <inertia
+        ixx="0.000224202818963409"
+        ixy="-1.96773409840189E-13"
+        ixz="-2.99224798427881E-05"
+        iyy="0.000286616921839535"
+        iyz="-3.10964171549742E-13"
+        izz="0.000349957607258242" />
+    </inertial>
   </link>
   <link name="l1_link">
@@ -40,7 +52,18 @@
       <origin rpy="0 0 0" xyz="0 0 0"/>
     </collision>
-    <xacro:inertial_cylinder mass="0.5" radius="0.03" length="0.05">
-      <origin xyz="0 0 0" rpy="0 0 0"/>
-    </xacro:inertial_cylinder>
+    <inertial>
+      <origin
+        xyz="-3.11559626639357E-12 9.70240468164796E-06 -0.0146667419724465"
+        rpy="0 0 0" />
+      <mass
+        value="0.0928887601998397" />
+      <inertia
+        ixx="6.09210980255232E-05"
+        ixy="-2.79207542479444E-18"
+        ixz="4.24841739939559E-15"
+        iyy="2.53493566630784E-05"
+        iyz="2.16442830142331E-08"
+        izz="4.88050835919342E-05" />
+    </inertial>
   </link>
   <link name="l2_link">
@@ -58,7 +81,18 @@
       <origin rpy="0 0 0" xyz="0 0 -0.03796"/>
     </collision>
-    <xacro:inertial_cylinder mass="0.5" radius="0.03" length="0.05">
-      <origin xyz="0 0 0" rpy="0 0 0"/>
-    </xacro:inertial_cylinder>
+    <inertial>
+      <origin
+        xyz="0.122021157535333 6.61338425981053E-05 -9.50311342843365E-05"
+        rpy="0 0 0" />
+      <mass
+        value="0.0895817175833772" />
+      <inertia
+        ixx="2.6269354271334E-05"
+        ixy="-2.55344668379587E-06"
+        ixz="-3.90237379833709E-09"
+        iyy="0.000350369536011831"
+        iyz="-6.82396195680563E-09"
+        izz="0.000333056833230846" />
+    </inertial>
   </link>
   <link name="l3_link">
@@ -76,7 +110,18 @@
       <origin rpy="0 0 0" xyz="-0.03 0 -0.27477"/>
     </collision>
-    <xacro:inertial_cylinder mass="0.5" radius="0.03" length="0.05">
-      <origin xyz="0 0 0" rpy="0 0 0"/>
-    </xacro:inertial_cylinder>
+    <inertial>
+      <origin
+        xyz="-0.00076280945740961 -0.114419656440929 -0.000177274968057332"
+        rpy="0 0 0" />
+      <mass
+        value="0.123009044986454" />
+      <inertia
+        ixx="0.000104111883333949"
+        ixy="1.06443789581137E-07"
+        ixz="1.54925816846055E-07"
+        iyy="1.46357151076022E-05"
+        iyz="-1.6435520156444E-07"
+        izz="0.000104009297710106" />
+    </inertial>
   </link>
   <link name="l4_link">
@@ -94,7 +139,18 @@
       <origin rpy="0 0 0" xyz="-0.03 0 -0.49076"/>
     </collision>
-    <xacro:inertial_cylinder mass="0.5" radius="0.03" length="0.05">
-      <origin xyz="0 0 0" rpy="0 0 0"/>
-    </xacro:inertial_cylinder>
+    <inertial>
+      <origin
+        xyz="0.0288857415118809 -0.000776842039187049 -0.000779764534254559"
+        rpy="0 0 0" />
+      <mass
+        value="0.00365697683069397" />
+      <inertia
+        ixx="1.15139272656909E-06"
+        ixy="1.31250385773157E-07"
+        ixz="-2.41954534039415E-13"
+        iyy="2.33034171341163E-06"
+        iyz="4.1392257505497E-13"
+        izz="1.47179863096272E-06" />
+    </inertial>
   </link>
   <joint name="base_to_L1" type="revolute">

File: roarm/urdf/robot.urdf.xacro (robot description, xacro)
@@ -2,4 +2,4 @@
 <robot xmlns:xacro="http://www.ros.org/wiki/xacro" name="robot">
     <xacro:include filename="roarm.xacro"/>
-    <!--xacro:include filename="ros2_control.xacro"/-->
+    <xacro:include filename="ros2_control.xacro"/>
 </robot>

File: roarm/urdf/ros2_control.xacro (robot description, xacro)
@@ -5,4 +5,56 @@
             <plugin>ign_ros2_control/IgnitionSystem</plugin>
         </hardware>
+        <joint name="base_to_L1">
+            <command_interface name="position">
+                <param name="min">-1000</param>
+                <param name="max">1000</param>
+            </command_interface>
+            <command_interface name="velocity">
+                <param name="min">-1000</param>
+                <param name="max">1000</param>
+            </command_interface>
+            <state_interface name="position"/>
+            <state_interface name="velocity"/>
+            <state_interface name="effort"/>
+        </joint>
+        <joint name="L1_to_L2">
+            <command_interface name="position">
+                <param name="min">-1000</param>
+                <param name="max">1000</param>
+            </command_interface>
+            <command_interface name="velocity">
+                <param name="min">-1000</param>
+                <param name="max">1000</param>
+            </command_interface>
+            <state_interface name="position"/>
+            <state_interface name="velocity"/>
+            <state_interface name="effort"/>
+        </joint>
+        <joint name="L2_to_L3">
+            <command_interface name="position">
+                <param name="min">-1000</param>
+                <param name="max">1000</param>
+            </command_interface>
+            <command_interface name="velocity">
+                <param name="min">-1000</param>
+                <param name="max">1000</param>
+            </command_interface>
+            <state_interface name="position"/>
+            <state_interface name="velocity"/>
+            <state_interface name="effort"/>
+        </joint>
+        <joint name="L3_to_L4">
+            <command_interface name="position">
+                <param name="min">-1000</param>
+                <param name="max">1000</param>
+            </command_interface>
+            <command_interface name="velocity">
+                <param name="min">-1000</param>
+                <param name="max">1000</param>
+            </command_interface>
+            <state_interface name="position"/>
+            <state_interface name="velocity"/>
+            <state_interface name="effort"/>
+        </joint>
     </ros2_control>
     <gazebo>

Commit message: Add most recent urdf updates

File: roarm/urdf/roarm.xacro (robot description, xacro)
@@ -1,184 +1,146 @@
 <?xml version="1.0"?>
 <robot xmlns:xacro="http://www.ros.org/wiki/xacro">
-  <material name="gray">
-    <color rgba="0.8 0.8 0.8 1"/>
-  </material>
-  <material name="white">
-    <color rgba="1 1 1 1"/>
-  </material>
-  <!--For now, set the inertial values according to here https://github.com/waveshareteam/roarm_ws_em0-->
-  <!--The current values are for the gripper layout roarm m2-->
+  <xacro:include filename="materials.xacro"/>
+  <link name="world"></link>
   <link name="base_link">
-    <visual>
-      <geometry>
-        <mesh filename="package://roarm/meshes/base.stl"/>
-      </geometry>
-      <origin rpy="0 0 0" xyz="0 0 0"/>
-      <material name="gray"/>
-    </visual>
-    <collision>
-      <geometry>
-        <mesh filename="package://roarm/meshes/base.stl"/>
-      </geometry>
-      <origin rpy="0 0 0" xyz="0 0 0"/>
-    </collision>
-    <inertial>
-      <origin
-        xyz="0.00373847392098165 -1.52445893424664E-10 0.0264265327292804"
-        rpy="0 0 0" />
-      <mass
-        value="0.326392759093976" />
-      <inertia
-        ixx="0.000224202818963409"
-        ixy="-1.96773409840189E-13"
-        ixz="-2.99224798427881E-05"
-        iyy="0.000286616921839535"
-        iyz="-3.10964171549742E-13"
-        izz="0.000349957607258242" />
-    </inertial>
-  </link>
-  <link name="l1_link">
-    <visual>
-      <geometry>
-        <mesh filename="package://roarm/meshes/L1.stl"/>
-      </geometry>
-      <origin rpy="0 0 0" xyz="0 0 0"/>
-      <material name="white"/>
-    </visual>
-    <collision>
-      <geometry>
-        <mesh filename="package://roarm/meshes/L1.stl"/>
-      </geometry>
-      <origin rpy="0 0 0" xyz="0 0 0"/>
-    </collision>
-    <inertial>
-      <origin
-        xyz="-3.11559626639357E-12 9.70240468164796E-06 -0.0146667419724465"
-        rpy="0 0 0" />
-      <mass
-        value="0.0928887601998397" />
-      <inertia
-        ixx="6.09210980255232E-05"
-        ixy="-2.79207542479444E-18"
-        ixz="4.24841739939559E-15"
-        iyy="2.53493566630784E-05"
-        iyz="2.16442830142331E-08"
-        izz="4.88050835919342E-05" />
-    </inertial>
-  </link>
-  <link name="l2_link">
-    <visual>
-      <geometry>
-        <mesh filename="package://roarm/meshes/L2.stl"/>
-      </geometry>
-      <origin rpy="0 0 0" xyz="0 0 -0.03796"/>
-      <material name="white"/>
-    </visual>
-    <collision>
-      <geometry>
-        <mesh filename="package://roarm/meshes/L2.stl"/>
-      </geometry>
-      <origin rpy="0 0 0" xyz="0 0 -0.03796"/>
-    </collision>
-    <inertial>
-      <origin
-        xyz="0.122021157535333 6.61338425981053E-05 -9.50311342843365E-05"
-        rpy="0 0 0" />
-      <mass
-        value="0.0895817175833772" />
-      <inertia
-        ixx="2.6269354271334E-05"
-        ixy="-2.55344668379587E-06"
-        ixz="-3.90237379833709E-09"
-        iyy="0.000350369536011831"
-        iyz="-6.82396195680563E-09"
-        izz="0.000333056833230846" />
-    </inertial>
-  </link>
-  <link name="l3_link">
-    <visual>
-      <geometry>
-        <mesh filename="package://roarm/meshes/L3.stl"/>
-      </geometry>
-      <origin rpy="0 0 0" xyz="-0.03 0 -0.27477"/>
-      <material name="white"/>
-    </visual>
-    <collision>
-      <geometry>
-        <mesh filename="package://roarm/meshes/L3.stl"/>
-      </geometry>
-      <origin rpy="0 0 0" xyz="-0.03 0 -0.27477"/>
-    </collision>
-    <inertial>
-      <origin
-        xyz="-0.00076280945740961 -0.114419656440929 -0.000177274968057332"
-        rpy="0 0 0" />
-      <mass
-        value="0.123009044986454" />
-      <inertia
-        ixx="0.000104111883333949"
-        ixy="1.06443789581137E-07"
-        ixz="1.54925816846055E-07"
-        iyy="1.46357151076022E-05"
-        iyz="-1.6435520156444E-07"
-        izz="0.000104009297710106" />
-    </inertial>
-  </link>
-  <link name="l4_link">
-    <visual>
-      <geometry>
-        <mesh filename="package://roarm/meshes/L4.stl"/>
-      </geometry>
-      <origin rpy="0 0 0" xyz="-0.03 0 -0.49076"/>
-      <material name="white"/>
-    </visual>
-    <collision>
-      <geometry>
-        <mesh filename="package://roarm/meshes/L4.stl"/>
-      </geometry>
-      <origin rpy="0 0 0" xyz="-0.03 0 -0.49076"/>
-    </collision>
-    <inertial>
-      <origin
-        xyz="0.0288857415118809 -0.000776842039187049 -0.000779764534254559"
-        rpy="0 0 0" />
-      <mass
-        value="0.00365697683069397" />
-      <inertia
-        ixx="1.15139272656909E-06"
-        ixy="1.31250385773157E-07"
-        ixz="-2.41954534039415E-13"
-        iyy="2.33034171341163E-06"
-        iyz="4.1392257505497E-13"
-        izz="1.47179863096272E-06" />
-    </inertial>
-  </link>
-  <joint name="base_to_L1" type="revolute">
-    <axis xyz="0 0 1"/>
-    <limit effort="1000.0" lower="-3.14" upper="3.14" velocity="0.5"/>
-    <parent link="base_link"/>
-    <child link="l1_link"/>
-    <origin xyz="0 0 0"/>
-  </joint>
-  <joint name="L1_to_L2" type="revolute">
-    <axis xyz="0 1 0"/>
-    <limit effort="1000.0" lower="-1.570796" upper="1.570796" velocity="0.5"/>
-    <parent link="l1_link"/>
-    <child link="l2_link"/>
-    <origin xyz="0 0 0.03796"/>
-  </joint>
-  <joint name="L2_to_L3" type="revolute">
-    <axis xyz="0 1 0"/>
-    <limit effort="1000.0" lower="-0.78539815" upper="3.1415926" velocity="0.5"/>
-    <parent link="l2_link"/>
-    <child link="l3_link"/>
-    <origin xyz="0.03 0 0.23682"/>
-  </joint>
-  <joint name="L3_to_L4" type="revolute">
-    <axis xyz="0 1 0"/>
-    <limit effort="1000.0" lower="-2.3561942" upper="2.3561942" velocity="0.5"/>
-    <parent link="l3_link"/>
-    <child link="l4_link"/>
-    <origin xyz="0 0 0.21599"/>
-  </joint>
+  <inertial>
+    <origin xyz="0.0032 0 0.04" rpy="0 0 0" />
+    <mass value="0.2562183" />
+    <inertia ixx="0.00029211" ixy="0" ixz="0" iyy="0.00035719" iyz="0" izz="0.000349421" />
+  </inertial>
+  <visual>
+    <origin xyz="0 0 0" rpy="0 0 0" />
+    <geometry>
+      <mesh filename="file://$(find roarm)/meshes/base_link.stl"  scale="1.0 1.0 1.0"/>
+    </geometry>
+    <material name="silver"/>
+  </visual>
+  <collision>
+    <origin xyz="0 0 0" rpy="0 0 0" />
+    <geometry>
+      <mesh filename="file://$(find roarm)/meshes/base_link.stl"  scale="1.0 1.0 1.0"/>
+    </geometry>
+  </collision>
+</link>
+<link name="link1">
+  <inertial>
+    <origin xyz="0 0 -0.015" rpy="0 0 0" />
+    <mass value="0.0729177" />
+    <inertia ixx="4.68465E-05" ixy="0" ixz="0" iyy="3.32107E-05" iyz="0" izz="5.01023E-05" />
+  </inertial>
+  <visual>
+    <origin xyz="0 0 0" rpy="0 0 0" />
+    <geometry>
+      <mesh filename="file://$(find roarm)/meshes/link1.stl"  scale="1.0 1.0 1.0"/>
+    </geometry>
+    <material name="silver"/>
+  </visual>
+  <collision>
+    <origin xyz="0 0 0" rpy="0 0 0" />
+    <geometry>
+      <mesh filename="file://$(find roarm)/meshes/link1.stl"  scale="1.0 1.0 1.0"/>
+    </geometry>
+  </collision>
+</link>
+<link name="link2">
+  <inertial>
+    <origin xyz="0.122 0 0" rpy="0 0 0" />
+    <mass value="0.0703216" />
+    <inertia ixx="5.46501E-05" ixy="0" ixz="0" iyy="0.000423091" iyz="0" izz="0.000404557" />
+  </inertial>
+  <visual>
+    <origin xyz="0 0 0" rpy="0 0 0" />
+    <geometry>
+      <mesh filename="file://$(find roarm)/meshes/link2.stl"  scale="1.0 1.0 1.0"/>
+    </geometry>
+    <material name="silver"/>
+  </visual>
+  <collision>
+    <origin xyz="0 0 0" rpy="0 0 0" />
+    <geometry>
+      <mesh filename="file://$(find roarm)/meshes/link2.stl"  scale="1.0 1.0 1.0"/>
+    </geometry>
+  </collision>
+</link>
+<link name="link3">
+  <inertial>
+    <origin xyz="0.002 -0.13687 0.0059" rpy="0 0 0" />
+    <mass value="0.0269773" />
+    <inertia ixx="0.000199591" ixy="0" ixz="0" iyy="8.01674E-06" iyz="0" izz="0.000196918" />
+  </inertial>
+  <visual>
+    <origin xyz="0 0 0" rpy="0 0 0" />
+    <geometry>
+      <mesh filename="file://$(find roarm)/meshes/link3.stl"  scale="1.0 1.0 1.0"/>
+    </geometry>
+    <material name="silver"/>
+  </visual>
+  <collision>
+    <origin xyz="0 0 0" rpy="0 0 0" />
+    <geometry>
+      <mesh filename="file://$(find roarm)/meshes/link3.stl"  scale="1.0 1.0 1.0"/>
+    </geometry>
+  </collision>
+</link>
+<link name="gripper_link">
+  <inertial>
+    <origin xyz="0.029 0.0027 -0.00078" rpy="0 0 0" />
+    <mass value="0.0028708" />
+    <inertia ixx="5.23216E-07" ixy="0" ixz="0" iyy="1.82071E-06" iyz="0" izz="1.60231E-06" />
+  </inertial>
+  <visual>
+    <origin xyz="0 0 0" rpy="0 0 0" />
+    <geometry>
+      <mesh filename="file://$(find roarm)/meshes/gripper_link.stl"  scale="1.0 1.0 1.0"/>
+    </geometry>
+    <material name="silver"/>
+  </visual>
+  <collision>
+    <origin xyz="0 0 0" rpy="0 0 0" />
+    <geometry>
+      <mesh filename="file://$(find roarm)/meshes/gripper_link.stl"  scale="1.0 1.0 1.0"/>
+    </geometry>
+  </collision>
+</link>
+<link name="hand_tcp"></link>
+<joint name="world_to_base_link" type="fixed">
+  <origin xyz="0.0 0.0 0.0" rpy="0 0 0"/>
+  <parent link="world"/>
+  <child link="base_link"/>
+  <axis xyz="0.0 0.0 1.0"/>
+</joint>
+<joint name="base_link_to_link1" type="revolute">
+  <origin xyz="0.0100000008759151 0 0.123059270461044" rpy="0 0 0" />
+  <parent link="base_link" />
+  <child link="link1" />
+  <axis xyz="0 0 1" />
+  <limit lower="-3.1416" upper="3.1416" effort="1000" velocity="0.5" />
+</joint>
+<joint name="link1_to_link2" type="revolute">
+  <origin xyz="0 0 0" rpy="-1.5708 -1.5708 0" />
+  <parent link="link1" />
+  <child link="link2" />
+  <axis xyz="0 0 1" />
+  <limit lower="-1.5708" upper="1.5708" effort="1000" velocity="0.5" />
+</joint>
+<joint name="link2_to_link3" type="revolute">
+  <origin xyz="0.236815132922094 0.0300023995170449 0" rpy="0 0 1.5708" />
+  <parent link="link2" />
+  <child  link="link3" />
+  <axis xyz="0 0 1" />
+  <limit lower="-1" upper="2.95" effort="1000" velocity="0.5" />
+</joint>
+<joint name="link3_to_gripper_link" type="revolute">
+  <origin xyz="0.002906 -0.21599 -0.00066683" rpy="-1.5708 0 -1.5708" />
+  <parent link="link3" />
+  <child link="gripper_link" />
+  <axis xyz="0 0 1" />
+  <limit lower="0" upper="1.5" effort="1000" velocity="0.5" />
+</joint>
+<joint name="link3_to_hand_tcp" type="fixed">
+  <origin xyz="0.002 -0.2802 0" rpy="1.5708 0 -1.5708" />
+  <parent link="link3" />
+  <child link="hand_tcp" />
+  <axis xyz="0 0 0" />
+</joint>
 </robot>

File: roarm/urdf/ros2_control.xacro (robot description, xacro)
@@ -5,5 +5,5 @@
             <plugin>gz_ros2_control/GazeboSimSystem</plugin>
         </hardware>
-        <joint name="base_to_L1">
+        <joint name="base_link_to_link1">
             <command_interface name="position">
                 <param name="min">-1000</param>
@@ -18,5 +18,5 @@
             <state_interface name="effort"/>
         </joint>
-        <joint name="L1_to_L2">
+        <joint name="link1_to_link2">
             <command_interface name="position">
                 <param name="min">-1000</param>
@@ -31,5 +31,5 @@
             <state_interface name="effort"/>
         </joint>
-        <joint name="L2_to_L3">
+        <joint name="link2_to_link3">
             <command_interface name="position">
                 <param name="min">-1000</param>
@@ -44,5 +44,5 @@
             <state_interface name="effort"/>
         </joint>
-        <joint name="L3_to_L4">
+        <joint name="link3_to_gripper_link">
             <command_interface name="position">
                 <param name="min">-1000</param>

Commit message: Change original urdf to gripper configuration

File: roarm/urdf/roarm.xacro (robot description, xacro)
@@ -176,5 +176,5 @@
   </joint>
   <joint name="L3_to_L4" type="revolute">
-    <axis xyz="0 1 0"/>
+    <axis xyz="-1 0 0"/>
     <limit effort="1000.0" lower="-2.3561942" upper="2.3561942" velocity="0.5"/>
     <parent link="l3_link"/>
