Commit message: Rename roarm package to roarm description

File: roarm_description/urdf/roarm.xacro (robot description, xacro)
@@ -11,5 +11,5 @@
       <origin xyz="0 0 0" rpy="0 0 0" />
       <geometry>
-        <mesh filename="file://$(find roarm)/meshes/base_link.stl"  scale="1.0 1.0 1.0"/>
+        <mesh filename="file://$(find roarm_description)/meshes/base_link.stl"  scale="1.0 1.0 1.0"/>
       </geometry>
       <material name="silver"/>
@@ -18,5 +18,5 @@
       <origin xyz="0 0 0" rpy="0 0 0" />
       <geometry>
-        <mesh filename="file://$(find roarm)/meshes/base_link.stl"  scale="1.0 1.0 1.0"/>
+        <mesh filename="file://$(find roarm_description)/meshes/base_link.stl"  scale="1.0 1.0 1.0"/>
       </geometry>
     </collision>
@@ -31,5 +31,5 @@
       <origin xyz="0 0 0" rpy="0 0 0" />
       <geometry>
-        <mesh filename="file://$(find roarm)/meshes/link1.stl"  scale="1.0 1.0 1.0"/>
+        <mesh filename="file://$(find roarm_description)/meshes/link1.stl"  scale="1.0 1.0 1.0"/>
       </geometry>
       <material name="silver"/>
@@ -38,5 +38,5 @@
       <origin xyz="0 0 0" rpy="0 0 0" />
       <geometry>
-        <mesh filename="file://$(find roarm)/meshes/link1.stl"  scale="1.0 1.0 1.0"/>
+        <mesh filename="file://$(find roarm_description)/meshes/link1.stl"  scale="1.0 1.0 1.0"/>
       </geometry>
     </collision>
@@ -51,5 +51,5 @@
       <origin xyz="0 0 0" rpy="0 0 0" />
       <geometry>
-        <mesh filename="file://$(find roarm)/meshes/link2.stl"  scale="1.0 1.0 1.0"/>
+        <mesh filename="file://$(find roarm_description)/meshes/link2.stl"  scale="1.0 1.0 1.0"/>
       </geometry>
       <material name="silver"/>
@@ -58,5 +58,5 @@
       <origin xyz="0 0 0" rpy="0 0 0" />
       <geometry>
-        <mesh filename="file://$(find roarm)/meshes/link2.stl"  scale="1.0 1.0 1.0"/>
+        <mesh filename="file://$(find roarm_description)/meshes/link2.stl"  scale="1.0 1.0 1.0"/>
       </geometry>
     </collision>
@@ -71,5 +71,5 @@
       <origin xyz="0 0 0" rpy="0 0 0" />
       <geometry>
-        <mesh filename="file://$(find roarm)/meshes/link3.stl"  scale="1.0 1.0 1.0"/>
+        <mesh filename="file://$(find roarm_description)/meshes/link3.stl"  scale="1.0 1.0 1.0"/>
       </geometry>
       <material name="silver"/>
@@ -78,5 +78,5 @@
       <origin xyz="0 0 0" rpy="0 0 0" />
       <geometry>
-        <mesh filename="file://$(find roarm)/meshes/link3.stl"  scale="1.0 1.0 1.0"/>
+        <mesh filename="file://$(find roarm_description)/meshes/link3.stl"  scale="1.0 1.0 1.0"/>
       </geometry>
     </collision>
@@ -91,5 +91,5 @@
       <origin xyz="0 0 0" rpy="0 0 0" />
       <geometry>
-        <mesh filename="file://$(find roarm)/meshes/gripper_link.stl"  scale="1.0 1.0 1.0"/>
+        <mesh filename="file://$(find roarm_description)/meshes/gripper_link.stl"  scale="1.0 1.0 1.0"/>
       </geometry>
       <material name="silver"/>
@@ -98,5 +98,5 @@
       <origin xyz="0 0 0" rpy="0 0 0" />
       <geometry>
-        <mesh filename="file://$(find roarm)/meshes/gripper_link.stl"  scale="1.0 1.0 1.0"/>
+        <mesh filename="file://$(find roarm_description)/meshes/gripper_link.stl"  scale="1.0 1.0 1.0"/>
       </geometry>
     </collision>

File: roarm_description/urdf/ros2_control.xacro (robot description, xacro)
@@ -62,5 +62,5 @@
             <robot_param>robot_description</robot_param>
             <robot_param_node>robot_state_publisher</robot_param_node>
-            <parameters>$(find roarm)/config/sim_controllers.yaml</parameters>
+            <parameters>$(find roarm_description)/config/sim_controllers.yaml</parameters>
         </plugin>
     </gazebo>

Commit message: Add publisher to controller topic

File: roarm_description/urdf/roarm.xacro (robot description, xacro)
@@ -108,5 +108,5 @@
     <child link="link1" />
     <axis xyz="0 0 1" />
-    <limit lower="-3.1416" upper="3.1416" effort="1000" velocity="0.5" />
+    <limit lower="-3.1416" upper="3.1416" effort="1000" velocity="1.0" />
   </joint>
   <joint name="link1_to_link2" type="revolute">
@@ -115,5 +115,5 @@
     <child link="link2" />
     <axis xyz="0 0 1" />
-    <limit lower="-1.5708" upper="1.5708" effort="1000" velocity="0.5" />
+    <limit lower="-1.5708" upper="1.5708" effort="1000" velocity="1.0" />
   </joint>
   <joint name="link2_to_link3" type="revolute">
@@ -122,5 +122,5 @@
     <child  link="link3" />
     <axis xyz="0 0 1" />
-    <limit lower="-1" upper="2.95" effort="1000" velocity="0.5" />
+    <limit lower="-1" upper="2.95" effort="1000" velocity="1.0" />
   </joint>
   <joint name="link3_to_gripper_link" type="revolute">
@@ -129,5 +129,5 @@
     <child link="gripper_link" />
     <axis xyz="0 0 1" />
-    <limit lower="0" upper="1.5" effort="1000" velocity="0.5" />
+    <limit lower="0" upper="1.5" effort="1000" velocity="1.0" />
   </joint>
   <joint name="link3_to_hand_tcp" type="fixed">

File: roarm_description/urdf/ros2_control.xacro (robot description, xacro)
@@ -62,5 +62,5 @@
             <robot_param>robot_description</robot_param>
             <robot_param_node>robot_state_publisher</robot_param_node>
-            <parameters>$(find roarm_description)/config/sim_controllers.yaml</parameters>
+            <parameters>$(find roarm_description)/config/test_controllers.yaml</parameters>
         </plugin>
     </gazebo>
